Commit message: support robotera_l7

File: assets/xbot_description/urdf/l7.urdf (robot description, URDF)
Before this commit: robot l7, 49 links, 48 joints
Links:
- link base_link: geometry visual mesh filename=../meshes/base_link.STL
- link left_ankle_pitch_link: geometry visual mesh filename=../meshes/left_ankle_pitch_link.STL
- link left_ankle_roll_link: geometry collision mesh filename=../meshes/left_ankle_roll_link.STL; visual mesh filename=../meshes/left_ankle_roll_link.STL
- link left_arm_base_link: geometry visual mesh filename=../meshes/left_arm_base_link.STL
- link left_arm_flange_link: geometry visual mesh filename=../meshes/left_arm_flange_link.STL
- link left_arm_yaw_link: geometry visual mesh filename=../meshes/left_arm_yaw_link.STL
- link left_elbow_pitch_link: geometry collision mesh filename=../meshes/left_elbow_pitch_link.STL; visual mesh filename=../meshes/left_elbow_pitch_link.STL
- link left_elbow_yaw_link: geometry collision mesh filename=../meshes/left_elbow_yaw_link.STL; visual mesh filename=../meshes/left_elbow_yaw_link.STL
- link left_hand_flange_link: geometry visual mesh filename=../meshes/left_hand_flange_link.STL
- link left_hip_pitch_link: geometry collision box size=0.1 0.06 0.15; visual mesh filename=../meshes/left_hip_pitch_link.STL
- link left_hip_roll_link: geometry collision mesh filename=../meshes/left_hip_roll_link.STL; visual mesh filename=../meshes/left_hip_roll_link.STL
- link left_hip_yaw_link: geometry collision cylinder length=0.16 radius=0.09; visual mesh filename=../meshes/left_hip_yaw_link.STL
- link left_knee_link: geometry collision mesh filename=../meshes/left_knee_link.STL; visual mesh filename=../meshes/left_knee_link.STL
- link left_shoulder_pitch_link: geometry collision mesh filename=../meshes/left_shoulder_pitch_link.STL; visual mesh filename=../meshes/left_shoulder_pitch_link.STL
- link left_shoulder_roll_link: geometry collision cylinder length=0.13 radius=0.045; visual mesh filename=../meshes/left_shoulder_roll_link.STL
- link left_wrist_pitch_link: geometry visual mesh filename=../meshes/left_wrist_pitch_link.STL
- link left_wrist_roll_link: geometry collision cylinder length=0.015 radius=0.025; visual mesh filename=../meshes/left_wrist_roll_link.STL
- link lidar_link: geometry visual mesh filename=../meshes/lidar_link.STL
- link mic_link: geometry visual mesh filename=../meshes/mic_link.STL
- link neck_base_link: geometry visual mesh filename=../meshes/neck_base_link.STL
- link neck_flange_link: geometry visual mesh filename=../meshes/neck_flange_link.STL
- link neck_pitch_link: geometry collision mesh filename=../meshes/neck_pitch_link.STL; visual mesh filename=../meshes/neck_pitch_link.STL
- link neck_yaw_link: geometry visual mesh filename=../meshes/neck_yaw_link.STL
- link right_ankle_pitch_link: geometry visual mesh filename=../meshes/right_ankle_pitch_link.STL
- link right_ankle_roll_link: geometry collision mesh filename=../meshes/right_ankle_roll_link.STL; visual mesh filename=../meshes/right_ankle_roll_link.STL
- link right_arm_base_link: geometry visual mesh filename=../meshes/right_arm_base_link.STL
- link right_arm_flange_link: geometry visual mesh filename=../meshes/right_arm_flange_link.STL
- link right_arm_yaw_link: geometry visual mesh filename=../meshes/right_arm_yaw_link.STL
- link right_elbow_pitch_link: geometry collision mesh filename=../meshes/right_elbow_pitch_link.STL; visual mesh filename=../meshes/right_elbow_pitch_link.STL
- link right_elbow_yaw_link: geometry collision mesh filename=../meshes/right_elbow_yaw_link.STL; visual mesh filename=../meshes/right_elbow_yaw_link.STL
- link right_hand_flange_link: geometry visual mesh filename=../meshes/right_hand_flange_link.STL
- link right_hip_pitch_link: geometry collision box size=0.1 0.06 0.15; visual mesh filename=../meshes/right_hip_pitch_link.STL
- link right_hip_roll_link: geometry collision mesh filename=../meshes/right_hip_roll_link.STL; visual mesh filename=../meshes/right_hip_roll_link.STL
- link right_hip_yaw_link: geometry collision cylinder length=0.16 radius=0.09; visual mesh filename=../meshes/right_hip_yaw_link.STL
- link right_knee_link: geometry collision mesh filename=../meshes/right_knee_link.STL; visual mesh filename=../meshes/right_knee_link.STL
- link right_shoulder_pitch_link: geometry collision mesh filename=../meshes/right_shoulder_pitch_link.STL; visual mesh filename=../meshes/right_shoulder_pitch_link.STL
- link right_shoulder_roll_link: geometry collision cylinder length=0.13 radius=0.045; visual mesh filename=../meshes/right_shoulder_roll_link.STL
- link right_wrist_pitch_link: geometry visual mesh filename=../meshes/right_wrist_pitch_link.STL
- link right_wrist_roll_link: geometry collision cylinder length=0.015 radius=0.025; visual mesh filename=../meshes/right_wrist_roll_link.STL
- link stereo_link: geometry visual mesh filename=../meshes/stereo_link.STL
- link torso_base_link: geometry collision mesh filename=../meshes/torso_base_link.STL; visual mesh filename=../meshes/torso_base_link.STL
- link torso_flange_link: geometry visual mesh filename=../meshes/torso_flange_link.STL
- link waist_base_link: geometry visual mesh filename=../meshes/waist_base_link.STL
- link waist_flange_link: geometry visual mesh filename=../meshes/waist_flange_link.STL
- link waist_pitch_link: geometry visual mesh filename=../meshes/waist_pitch_link.STL
- link waist_roll_link: geometry visual mesh filename=../meshes/waist_roll_link.STL
- link waist_yaw_link: geometry visual mesh filename=../meshes/waist_yaw_link.STL
